File: Hardware/LED Helper/LED Helper.sch (KiCad schematic (older format))
At the start: 18 parts, among them J1 Conn_01x10, J2 Conn_01x10

Commit message: Prepare for production
Parts:
- D1, D2, D3, D4, D5, D6, D7, D8: LCSC (none) -> C2293
- R1, R2, R3, R4, R5, R6, R7, R8: LCSC (none) -> C17630
Changed lines of the file:
@@
 F 2 "LED_SMD:LED_0805_2012Metric" H 3550 4700 50  0001 C CNN
 F 3 "~" H 3550 4700 50  0001 C CNN
+F 4 "C2293" H 3550 4700 50  0001 C CNN "LCSC"
 	1    3550 4700
 	0    -1   -1   0
@@
 F 2 "LED_SMD:LED_0805_2012Metric" H 4050 4700 50  0001 C CNN
 F 3 "~" H 4050 4700 50  0001 C CNN
+F 4 "C2293" H 4050 4700 50  0001 C CNN "LCSC"
 	1    4050 4700
 	0    -1   -1   0
@@
 F 2 "LED_SMD:LED_0805_2012Metric" H 4550 4700 50  0001 C CNN
 F 3 "~" H 4550 4700 50  0001 C CNN
+F 4 "C2293" H 4550 4700 50  0001 C CNN "LCSC"
 	1    4550 4700
 	0    -1   -1   0
@@
 F 2 "LED_SMD:LED_0805_2012Metric" H 5050 4700 50  0001 C CNN
 F 3 "~" H 5050 4700 50  0001 C CNN
+F 4 "C2293" H 5050 4700 50  0001 C CNN "LCSC"
 	1    5050 4700
 	0    -1   -1   0
@@
 F 2 "LED_SMD:LED_0805_2012Metric" H 5550 4700 50  0001 C CNN
 F 3 "~" H 5550 4700 50  0001 C CNN
+F 4 "C2293" H 5550 4700 50  0001 C CNN "LCSC"
 	1    5550 4700
 	0    -1   -1   0
@@
 F 2 "LED_SMD:LED_0805_2012Metric" H 6050 4700 50  0001 C CNN
 F 3 "~" H 6050 4700 50  0001 C CNN
+F 4 "C2293" H 6050 4700 50  0001 C CNN "LCSC"
 	1    6050 4700
 	0    -1   -1   0
@@
 F 2 "LED_SMD:LED_0805_2012Metric" H 6550 4700 50  0001 C CNN
 F 3 "~" H 6550 4700 50  0001 C CNN
+F 4 "C2293" H 6550 4700 50  0001 C CNN "LCSC"
 	1    6550 4700
 	0    -1   -1   0
@@
 F 2 "LED_SMD:LED_0805_2012Metric" H 7050 4700 50  0001 C CNN
 F 3 "~" H 7050 4700 50  0001 C CNN
+F 4 "C2293" H 7050 4700 50  0001 C CNN "LCSC"
 	1    7050 4700
 	0    -1   -1   0
@@
 F 2 "Resistor_SMD:R_0805_2012Metric" V 3480 5150 50  0001 C CNN
 F 3 "~" H 3550 5150 50  0001 C CNN
+F 4 "C17630" H 3550 5150 50  0001 C CNN "LCSC"
 	1    3550 5150
 	1    0    0    -1
@@
 F 2 "Resistor_SMD:R_0805_2012Metric" V 3980 5150 50  0001 C CNN
 F 3 "~" H 4050 5150 50  0001 C CNN
+F 4 "C17630" H 4050 5150 50  0001 C CNN "LCSC"
 	1    4050 5150
 	1    0    0    -1
@@
 F 2 "Resistor_SMD:R_0805_2012Metric" V 4480 5150 50  0001 C CNN
 F 3 "~" H 4550 5150 50  0001 C CNN
+F 4 "C17630" H 4550 5150 50  0001 C CNN "LCSC"
 	1    4550 5150
 	1    0    0    -1
@@
 F 2 "Resistor_SMD:R_0805_2012Metric" V 4980 5150 50  0001 C CNN
 F 3 "~" H 5050 5150 50  0001 C CNN
+F 4 "C17630" H 5050 5150 50  0001 C CNN "LCSC"
 	1    5050 5150
 	1    0    0    -1
@@
 F 2 "Resistor_SMD:R_0805_2012Metric" V 5480 5150 50  0001 C CNN
 F 3 "~" H 5550 5150 50  0001 C CNN
+F 4 "C17630" H 5550 5150 50  0001 C CNN "LCSC"
 	1    5550 5150
 	1    0    0    -1
@@
 F 2 "Resistor_SMD:R_0805_2012Metric" V 5980 5150 50  0001 C CNN
 F 3 "~" H 6050 5150 50  0001 C CNN
+F 4 "C17630" H 6050 5150 50  0001 C CNN "LCSC"
 	1    6050 5150
 	1    0    0    -1
@@
 F 2 "Resistor_SMD:R_0805_2012Metric" V 6480 5150 50  0001 C CNN
 F 3 "~" H 6550 5150 50  0001 C CNN
+F 4 "C17630" H 6550 5150 50  0001 C CNN "LCSC"
 	1    6550 5150
 	1    0    0    -1
@@
 F 2 "Resistor_SMD:R_0805_2012Metric" V 6980 5150 50  0001 C CNN
 F 3 "~" H 7050 5150 50  0001 C CNN
+F 4 "C17630" H 7050 5150 50  0001 C CNN "LCSC"
 	1    7050 5150
 	1    0    0    -1
