File: Hardware/Switch Helper/Switch Helper.sch (KiCad schematic (older format))
At the start: 8 parts, among them J1 Conn_01x10, J2 Conn_01x10, SW1 SW_SPST, U1 SN74LVC1G14DBV

Commit message: Prepare for production
Parts:
- C1: JLCPCB C49678 -> (none); LCSC (none) -> C49678
- D1: JLCPCB C64898 -> (none); LCSC (none) -> C64898
- R1, R2: JLCPCB C17414 -> (none); LCSC (none) -> C17414
- SW1: JLCPCB C318884 -> (none); LCSC (none) -> C318884
- U1: JLCPCB C7835 -> (none); LCSC (none) -> C7835
Changed lines of the file:
@@
 F 2 "Resistor_SMD:R_0805_2012Metric" V 6230 2500 50  0001 C CNN
 F 3 "~" H 6300 2500 50  0001 C CNN
-F 4 "C17414" H 6300 2500 50  0001 C CNN "JLCPCB"
+F 4 "C17414" H 6300 2500 50  0001 C CNN "LCSC"
 	1    6300 2500
 	1    0    0    -1
@@
 F 2 "Resistor_SMD:R_0805_2012Metric" V 6680 3200 50  0001 C CNN
 F 3 "~" H 6750 3200 50  0001 C CNN
-F 4 "C17414" H 6750 3200 50  0001 C CNN "JLCPCB"
+F 4 "C17414" H 6750 3200 50  0001 C CNN "LCSC"
 	1    6750 3200
 	0    1    1    0
@@
 F 2 "Diode_SMD:D_SOD-123F" H 6750 2850 50  0001 C CNN
 F 3 "~" H 6750 2850 50  0001 C CNN
-F 4 "C64898" H 6750 2850 50  0001 C CNN "JLCPCB"
+F 4 "C64898" H 6750 2850 50  0001 C CNN "LCSC"
 	1    6750 2850
 	-1   0    0    1
@@
 F 2 "Capacitor_SMD:C_0805_2012Metric" H 7238 3450 50  0001 C CNN
 F 3 "~" H 7200 3600 50  0001 C CNN
-F 4 "C49678" H 7200 3600 50  0001 C CNN "JLCPCB"
+F 4 "C49678" H 7200 3600 50  0001 C CNN "LCSC"
 	1    7200 3600
 	1    0    0    -1
@@
 F 2 "Switch Helper:SW_TS-1187A-B-A-B" H 6300 3550 50  0001 C CNN
 F 3 "~" H 6300 3550 50  0001 C CNN
-F 4 "C318884" V 6300 3550 50  0001 C CNN "JLCPCB"
+F 4 "C318884" V 6300 3550 50  0001 C CNN "LCSC"
 	1    6300 3550
 	0    -1   -1   0
@@
 F 2 "Package_TO_SOT_SMD:SOT-23-5" H 7750 2950 50  0001 C CNN
 F 3 "http://www.ti.com/lit/ds/symlink/sn74lvc1g14.pdf" H 7750 3200 50  0001 C CNN
-F 4 "C7835" H 7750 3200 50  0001 C CNN "JLCPCB"
+F 4 "C7835" H 7750 3200 50  0001 C CNN "LCSC"
 	1    7750 3200
 	1    0    0    -1
